Commit message: update | 29 oct 2024, gazebo compatible ver.

File: urdf/first_robot.urdf (robot description, URDF)
Before this commit: robot Panzerkampfwagen VI Ausführung E, 3 links, 8 joints
Links:
- removed link base_link

File: urdf/shape_creator.xacro (robot description, xacro)
@@ -2,5 +2,6 @@
 <robot xmlns:xacro="http://ros.org/wiki/xacro">
     <xacro:include filename="generic_properties.xacro"/>
-    <xacro:macro name="cylinder_preset" params="prefix radius length xyz rpy material">
+    <xacro:include filename="inertia_calculator.xacro"/>
+    <xacro:macro name="cylinder_preset" params="prefix mass radius length xyz rpy material">
         <link name="${prefix}_link">
             <visual>
@@ -9,7 +10,12 @@
                 <material name="${material}"/>
             </visual>
+            <collision>
+                <origin xyz="${xyz}" rpy="${rpy}"/>
+                <geometry> <cylinder radius="${radius}" length="${length}"/> </geometry>
+            </collision>
+            <xacro:cylinder_inertia_calculator m="${mass}" r="${radius}" h="${length}" xyz="${xyz}" rpy="${rpy}"/>
         </link>
     </xacro:macro>
-    <xacro:macro name="cylinder_rgba" params="prefix radius length xyz rpy rgba">
+    <xacro:macro name="cylinder_rgba" params="prefix radius mass length xyz rpy rgba">
         <link name="${prefix}_link">
             <visual>
@@ -20,4 +26,39 @@
                 </material>
             </visual>
+            <collision>
+                <origin xyz="${xyz}" rpy="${rpy}"/>
+                <geometry> <cylinder radius="${radius}" length="${length}"/> </geometry>
+            </collision>
+            <xacro:cylinder_inertia_calculator m="${mass}" r="${radius}" h="${length}" xyz="${xyz}" rpy="${rpy}"/>
+        </link>
+    </xacro:macro>
+    <xacro:macro name="boxoid_preset" params="prefix mass length depth height xyz rpy material">
+        <link name="${prefix}_link">
+            <visual>
+                <origin xyz="${xyz}" rpy="${rpy}"/>
+                <geometry> <box size="${length} ${depth} ${height}"/> </geometry>
+                <material name="${material}"/>
+            </visual>
+            <collision>
+                <origin xyz="${xyz}" rpy="${rpy}"/>
+                <geometry> <box size="${length} ${depth} ${height}"/> </geometry>
+            </collision>
+            <xacro:boxoid_inertia_calculator m="${mass}" l="${length}" w="${depth}" h="${height}" xyz="${xyz}" rpy="${rpy}"/>
+        </link>
+    </xacro:macro>
+    <xacro:macro name="boxoid_rgba" params="prefix mass length depth height xyz rpy rgba">
+        <link name="${prefix}_link">
+            <visual>
+                <origin xyz="${xyz}" rpy="${rpy}"/>
+                <geometry> <box size="${length} ${depth} ${height}"/> </geometry>
+                <material name="ARCIBI">
+                    <color rgba="${rgba}"/>
+                </material>
+            </visual>
+            <collision>
+                <origin xyz="${xyz}" rpy="${rpy}"/>
+                <geometry> <box size="${length} ${depth} ${height}"/> </geometry>
+            </collision>
+            <xacro:boxoid_inertia_calculator m="${mass}" l="${length}" w="${depth}" h="${height}" xyz="${xyz}" rpy="${rpy}"/>
         </link>
     </xacro:macro>
