Commit message: update | 20 dec 2024, bug fixes and improvement on Gazebo sim

File: urdf/inertia_calculator.xacro (robot description, xacro)
@@ -1,23 +1,23 @@
 <?xml version="1.0"?>
 <robot xmlns:xacro="http://ros.org/wiki/xacro">
-    <xacro:macro name="boxoid_inertia_calculator" params="m l w h xyz rpy">
+    <xacro:macro name="box_inertia" params="m l w h xyz rpy">
         <inertial>
             <origin xyz="${xyz}" rpy="${rpy}"/>
             <mass value="${m}"/>
             <inertia ixx="${(m/12) * (h*h + l*l)}" ixy="0" ixz="0"
-                    iyy="${(m/12) * (w*w + l*l)}" iyx=""  iyz="0"
-                    izz="${(m/12) * (h*h + w*w)}" izx="0" izy="0"/>
+                    iyy="${(m/12) * (w*w + l*l)}" iyx="0"  iyz="0"
+                    izz="${(m/12) * (h*h + w*w)}" izx="0" izy="0" />
         </inertial>
     </xacro:macro>
-    <xacro:macro name="cylinder_inertia_calculator" params="m r h xyz rpy">
+    <xacro:macro name="cylinder_inertia" params="m r h xyz rpy">
         <inertial>
             <origin xyz="${xyz}" rpy="${rpy}" />
             <mass value="${m}" />
             <inertia ixx="${(m/12) * (3*r*r + h*h)}" ixy="0" ixz="0"
-                     iyy="${(m/12) * (3*r*r + h*h)}" iyz="0"
-                     izz="${(m/2) * (r*r)}" />
+                     iyy="${(m/12) * (3*r*r + h*h)}" iyx="0" iyz="0"
+                     izz="${(m/2) * (r*r)}"         izx="0" izy="0" />
         </inertial>
     </xacro:macro>
-    <xacro:macro name="sphere_inertia_calculator" params="m r xyz rpy">
+    <xacro:macro name="sphere_inertia" params="m r xyz rpy">
         <inertial>
             <origin xyz="${xyz}" rpy="${rpy}" />

File: urdf/shape_creator.xacro (robot description, xacro)
@@ -14,5 +14,5 @@
                 <geometry> <cylinder radius="${radius}" length="${length}"/> </geometry>
             </collision>
-            <xacro:cylinder_inertia_calculator m="${mass}" r="${radius}" h="${length}" xyz="${xyz}" rpy="${rpy}"/>
+            <xacro:cylinder_inertia m="${mass}" r="${radius}" h="${length}" xyz="${xyz}" rpy="${rpy}"/>
         </link>
     </xacro:macro>
@@ -22,5 +22,5 @@
                 <origin xyz="${xyz}" rpy="${rpy}"/>
                 <geometry> <cylinder radius="${radius}" length="${length}"/> </geometry>
-                <material name="ARCIBI">
+                <material name="${prefix}_link_color">
                     <color rgba="${rgba}"/>
                 </material>
@@ -30,27 +30,27 @@
                 <geometry> <cylinder radius="${radius}" length="${length}"/> </geometry>
             </collision>
-            <xacro:cylinder_inertia_calculator m="${mass}" r="${radius}" h="${length}" xyz="${xyz}" rpy="${rpy}"/>
+            <xacro:cylinder_inertia m="${mass}" r="${radius}" h="${length}" xyz="${xyz}" rpy="${rpy}"/>
         </link>
     </xacro:macro>
-    <xacro:macro name="boxoid_preset" params="prefix mass length depth height xyz rpy material">
+    <xacro:macro name="box_preset" params="prefix mass length width height xyz rpy material">
         <link name="${prefix}_link">
             <visual>
                 <origin xyz="${xyz}" rpy="${rpy}"/>
-                <geometry> <box size="${length} ${depth} ${height}"/> </geometry>
+                <geometry> <box size="${length} ${width} ${height}"/> </geometry>
                 <material name="${material}"/>
             </visual>
             <collision>
                 <origin xyz="${xyz}" rpy="${rpy}"/>
-                <geometry> <box size="${length} ${depth} ${height}"/> </geometry>
+                <geometry> <box size="${length} ${width} ${height}"/> </geometry>
             </collision>
-            <xacro:boxoid_inertia_calculator m="${mass}" l="${length}" w="${depth}" h="${height}" xyz="${xyz}" rpy="${rpy}"/>
+            <xacro:box_inertia m="${mass}" l="${length}" w="${width}" h="${height}" xyz="${xyz}" rpy="${rpy}"/>
         </link>
     </xacro:macro>
-    <xacro:macro name="boxoid_rgba" params="prefix mass length depth height xyz rpy rgba">
+    <xacro:macro name="box_rgba" params="prefix mass length width height xyz rpy rgba">
         <link name="${prefix}_link">
             <visual>
                 <origin xyz="${xyz}" rpy="${rpy}"/>
-                <geometry> <box size="${length} ${depth} ${height}"/> </geometry>
-                <material name="ARCIBI">
+                <geometry> <box size="${length} ${width} ${height}"/> </geometry>
+                <material name="${prefix}_link_color">
                     <color rgba="${rgba}"/>
                 </material>
@@ -58,7 +58,23 @@
             <collision>
                 <origin xyz="${xyz}" rpy="${rpy}"/>
-                <geometry> <box size="${length} ${depth} ${height}"/> </geometry>
+                <geometry> <box size="${length} ${width} ${height}"/> </geometry>
             </collision>
-            <xacro:boxoid_inertia_calculator m="${mass}" l="${length}" w="${depth}" h="${height}" xyz="${xyz}" rpy="${rpy}"/>
+            <xacro:box_inertia m="${mass}" l="${length}" w="${width}" h="${height}" xyz="${xyz}" rpy="${rpy}"/>
+        </link>
+    </xacro:macro>
+    <xacro:macro name="sphere_rgba" params="prefix mass radius xyz rpy rgba">
+        <link name="${prefix}_link">
+            <visual>
+                <origin xyz="${xyz}" rpy="${rpy}"/>
+                <geometry> <sphere radius="${radius}"/> </geometry>
+                <material name="${prefix}_link_color">
+                    <color rgba="${rgba}"/>
+                </material>
+            </visual>
+            <collision>
+                <origin xyz="${xyz}" rpy="${rpy}"/>
+                <geometry> <sphere radius="${radius}"/> </geometry>
+            </collision>
+            <xacro:sphere_inertia m="${mass}" r="${radius}" xyz="${xyz}" rpy="${rpy}" />
         </link>
     </xacro:macro>
